File: pcb_class.sch (KiCad schematic (older format))
At the start: 10 parts, among them J1 Conn_01x04_Female, Q1 KSP13

Commit message: Footprints assigned, netlist generated
Parts:
- C1: footprint (none) -> Capacitor_THT:C_Disc_D9.0mm_W5.0mm_P7.50mm
- C2: footprint (none) -> Capacitor_THT:CP_Radial_D5.0mm_P2.00mm
- C3: value 100nF -> .1uF; footprint (none) -> Capacitor_THT:C_Rect_L7.2mm_W2.5mm_P5.00mm_FKS2_FKP2_MKS2_MKP2
- D1: footprint (none) -> Diode_THT:D_DO-35_SOD27_P7.62mm_Horizontal
- J1: footprint (none) -> Connector_PinSocket_2.54mm:PinSocket_1x04_P2.54mm_Vertical
- Q1: footprint (none) -> Package_TO_SOT_THT:TO-92_Inline
- R1: footprint (none) -> Resistor_THT:R_Axial_DIN0207_L6.3mm_D2.5mm_P10.16mm_Horizontal
- RV1, RV2, RV3: footprint (none) -> Connector_PinSocket_2.54mm:PinSocket_1x03_P2.54mm_Vertical
Changed lines of the file:
@@
 F 0 "R1" H 4070 2796 50  0000 L CNN
 F 1 "10K" H 4070 2705 50  0000 L CNN
-F 2 "" V 3930 2750 50  0001 C CNN
+F 2 "Resistor_THT:R_Axial_DIN0207_L6.3mm_D2.5mm_P10.16mm_Horizontal" V 3930 2750 50  0001 C CNN
 F 3 "~" H 4000 2750 50  0001 C CNN
 	1    4000 2750
@@
 P 4550 3000
 F 0 "C3" V 4802 3000 50  0000 C CNN
-F 1 "100nF" V 4711 3000 50  0000 C CNN
-F 2 "" H 4588 2850 50  0001 C CNN
+F 1 ".1uF" V 4711 3000 50  0000 C CNN
+F 2 "Capacitor_THT:C_Rect_L7.2mm_W2.5mm_P5.00mm_FKS2_FKP2_MKS2_MKP2" H 4588 2850 50  0001 C CNN
 F 3 "~" H 4550 3000 50  0001 C CNN
 	1    4550 3000
@@
 F 0 "D1" H 3750 3216 50  0000 C CNN
 F 1 "1N4148" H 3750 3125 50  0000 C CNN
-F 2 "" H 3750 3000 50  0001 C CNN
+F 2 "Diode_THT:D_DO-35_SOD27_P7.62mm_Horizontal" H 3750 3000 50  0001 C CNN
 F 3 "~" H 3750 3000 50  0001 C CNN
 	1    3750 3000
@@
 F 0 "RV3" H 5180 3396 50  0000 R CNN
 F 1 "A100K" H 5180 3305 50  0000 R CNN
-F 2 "" H 5250 3350 50  0001 C CNN
+F 2 "Connector_PinSocket_2.54mm:PinSocket_1x03_P2.54mm_Vertical" H 5250 3350 50  0001 C CNN
 F 3 "~" H 5250 3350 50  0001 C CNN
 	1    5250 3350
@@
 F 0 "Q1" H 4091 3346 50  0000 L CNN
 F 1 "KSP13" H 4091 3255 50  0000 L CNN
-F 2 "" H 4100 3400 50  0001 C CNN
+F 2 "Package_TO_SOT_THT:TO-92_Inline" H 4100 3400 50  0001 C CNN
 F 3 "~" H 3900 3300 50  0001 C CNN
 	1    3900 3300
@@
 F 0 "J1" H 2677 4226 50  0000 L CNN
 F 1 "Conn_01x04_Female" H 2677 4135 50  0000 L CNN
-F 2 "" H 2650 4250 50  0001 C CNN
+F 2 "Connector_PinSocket_2.54mm:PinSocket_1x04_P2.54mm_Vertical" H 2650 4250 50  0001 C CNN
 F 3 "~" H 2650 4250 50  0001 C CNN
 	1    2650 4250
@@
 F 0 "RV1" H 2730 3696 50  0000 R CNN
 F 1 "B100K" H 2730 3605 50  0000 R CNN
-F 2 "" H 2800 3650 50  0001 C CNN
+F 2 "Connector_PinSocket_2.54mm:PinSocket_1x03_P2.54mm_Vertical" H 2800 3650 50  0001 C CNN
 F 3 "~" H 2800 3650 50  0001 C CNN
 	1    2800 3650
@@
 F 0 "C2" V 2945 3900 50  0000 C CNN
 F 1 "2.2uF" V 3036 3900 50  0000 C CNN
-F 2 "" H 3238 3750 50  0001 C CNN
+F 2 "Capacitor_THT:CP_Radial_D5.0mm_P2.00mm" H 3238 3750 50  0001 C CNN
 F 3 "~" H 3200 3900 50  0001 C CNN
 	1    3200 3900
@@
 F 0 "C1" V 2948 3300 50  0000 C CNN
 F 1 "1nF" V 3039 3300 50  0000 C CNN
-F 2 "" H 3238 3150 50  0001 C CNN
+F 2 "Capacitor_THT:C_Disc_D9.0mm_W5.0mm_P7.50mm" H 3238 3150 50  0001 C CNN
 F 3 "~" H 3200 3300 50  0001 C CNN
 	1    3200 3300
@@
 F 0 "RV2" H 3930 3896 50  0000 R CNN
 F 1 "B1K" H 3930 3805 50  0000 R CNN
-F 2 "" H 4000 3850 50  0001 C CNN
+F 2 "Connector_PinSocket_2.54mm:PinSocket_1x03_P2.54mm_Vertical" H 4000 3850 50  0001 C CNN
 F 3 "~" H 4000 3850 50  0001 C CNN
 	1    4000 3850
